File: sch/atmel/encoder.kicad_pcb (KiCad board)
At the start: 2 copper layers, 100 x 100 mm, 69 parts, among them J1 GND-24V, J2 ENCODER, J3 ICSP, J4 CAN, Q1 BC817, Q2 MMBT2222A, U1 ATMEGA328P-PU, U2 DS1307, U3 LM7805CV, U4 PSW-8,5R, U5 PESD1CAN, U6 MPC2551, U7 MCP2515-E/SO, U8 MAX485CSA, Y1 16MHz, Y2 32.768KHz, Y3 16MHz

Commit message: placa endcoder
Routing:
- net GND: track 300.6 -> 471.7 mm, vias 7 -> 15
- net +5V: track 249.3 -> 368.4 mm, vias 8 -> 14
- net /TX: track 0.00 -> 91.5 mm, vias 0 -> 2
- net /LCD_D7: track 0.00 -> 74.3 mm, vias 0 -> 1
- net /LCD_D6: track 0.00 -> 71.0 mm, vias 0 -> 1
- net /LCD_D5: track 0.00 -> 68.3 mm, vias 0 -> 1
- net /PB3: track 0.00 -> 46.6 mm, vias 0 -> 3
- net /LCD_RS: track 0.00 -> 45.9 mm, vias 0 -> 2
- net /CAN_INT: track 0.00 -> 45.4 mm, vias 0 -> 4
- net /RX: track 0.00 -> 42.3 mm, vias 0 -> 2
- net /LCD_EN: track 0.00 -> 39.8 mm, vias 0 -> 2
- net /ENCODER_EN: track 0.00 -> 38.2 mm, vias 0 -> 2
- net /PB4: track 0.00 -> 38.1 mm, vias 0 -> 3
- net Net-(J2-Pad4): track 0.00 -> 33.8 mm
- net +BATT: track 0.00 -> 33.7 mm, vias 0 -> 1
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- added copper zone on B.Cu, net GND
- added copper zone on F.Cu, net GND

Commit message: lcd e heart_beat
Signed-off-by: cuki2 <mauricio@krebs.com.br>
Parts:
- added D8: RUN, w_smd_leds:Led_0805, F.Cu at (85.9, 80.8)
- added R21: 1k, w_smd_resistors:r_0805, F.Cu at (80.0, 80.8)
Connections:
- U1 pad 12: Net-(U1-Pad12) -> /CAN_RS
- U1 pad 13: /CAN_RS -> /HEART_BEAT
Routing:
- net /HEART_BEAT: track 0.00 -> 21.2 mm, vias 0 -> 2
- net /CAN_RS: track 12.5 -> 21.7 mm
- net Net-(D8-Pad1): track 0.00 -> 3.84 mm
- net Net-(D7-Pad2): track 72.1 -> 73.0 mm
