File: sch/microchip/microchip.sch (KiCad schematic (older format))
At the start: 65 parts

Commit message: Signed-off-by: cuki2 <mauricio@krebs.com.br>
Parts:
- added C12, C13: 22pF, w_smd_cap:c_0805, symbol C
- added C14, C15: 560pF, w_smd_cap:c_0805, symbol C
- added C16, C18: 100nF 50V, w_smd_cap:c_0805, symbol C
- added D3: CAN, w_smd_leds:Led_0805, symbol LED_AK
- added J2: ICSP, w_pin_strip:pin_strip_6, symbol CONN_01X06
- added J3: CAN, w_conn_mkds:mkds_1,5-2, symbol CONN_01X02
- added J5: SL1, w_conn_mkds:mkds_1,5-2, symbol CONN_01X02
- added R10, R12, R5: 100R, w_smd_resistors:r_0805, symbol R
- added R23: 4k7, w_smd_resistors:r_0805, symbol R
- added R32: 10k, w_smd_resistors:r_0805, symbol R
- added R6: 1k, w_smd_resistors:r_0805, symbol R
- added U5: MCP2515-E/SO, w_smd_dil:soic-18, symbol MCP2515-I/P
- added U6: PESD1CAN, w_smd_trans:sot23, symbol PESD1CAN
- added U7: MPC2551, w_smd_dil:so-8, symbol MPC2551
- added Y3: 16MHz, w_crystal:crystal_hc-49%2fsmd, symbol Crystal
- D10: renamed from D?; value RX -> RX1
- D7: renamed from D?; value TX -> TX2
- D8: renamed from D?; value TX -> TX1
- D9: renamed from D?; value RX -> RX2
- U1: renamed from U?; footprint (none) -> w_smd_qfn:qfn-28
- gave numbers to parts that had none: 60
Connections:
- net labels added: CAN_H, CAN_L, CAN_MISO, CAN_MOSI, RXD_CAN, TXD_CAN, XTAL5, XTAL6, ~MCLR
- net labels removed: A, B, PB3, PB4, RST
- wire segments 224 -> 283
- no-connect marks 5 -> 17
Other:
- moved on the sheet: C17, C19, D10, D4, D5, D6, D7, D8, D9, J4, Q1, Q2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

Commit message: Signed-off-by: cuki2 <mauricio@krebs.com.br>
Parts:
- added C20, C21: 100nF 50V, w_smd_cap:c_0805, symbol C
- added R33, R34: 10k, w_smd_resistors:r_0805, symbol R
- added SW1, SW2: SW_Push, w_switch:PCB_PUSH, symbol SW_Push
Connections:
- net +5V: now also R33.1, R34.1
- net +BATT: now also U1.24 (RB3/AN9/C12IN2-/CTED2/CCP2/P2A/SDO2); no longer U2.3 (Vbat)
- net GND: now also C20.2, C21.2, SW1.2, SW2.2
- net BTO1: now reaches U1.22 (RB1/AN10/C12IN3-/P1C/SCK2/SCL2/INT1)
- net BTO1: now also C20.1, R33.2, SW1.1
- net BTO2: now reaches U1.23 (RB2/AN8/CTED1/P1B/SDI2/SDA2/INT2)
- net BTO2: now also C21.1, R34.2, SW2.1
- no-connect marks 17 -> 14
Other:
- moved on the sheet: BT1, C1, C18, C2, C3, C5, C9, DS1, R1, R2, R23, R9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
