File: sch/microchip/microchip.kicad_pcb (KiCad board)
At the start: 2 copper layers, 100 x 100 mm, 85 parts, among them J1 GND-24V, J2 ICSP, J3 CAN, J4 ENCODER, J5 SL1, Q1 BC817, Q2 MMBT2222A, Q3 MMBT2222A, U1 PIC18(L)F2X/4XK22-P, U2 DS1307, U3 LD1117S50TR, U4 L7805CD2T, U5 MCP2515-E/SO, U6 PESD1CAN, U7 MPC2551, U8 MAX485CSA, U9 MAX485CSA, Y1 16MHz, Y2 32.768KHz, Y3 16MHz

Commit message: Signed-off-by: cuki2 <mauricio@krebs.com.br>
Parts:
- added C20: 100nF 50V, w_smd_cap:c_0805, B.Cu at (25.9, 97.0)
- added C21: 100nF 50V, w_smd_cap:c_0805, B.Cu at (36.1, 97.0)
- added R33: 10k, w_smd_resistors:r_0805, F.Cu at (23.6, 89.4)
- added R34: 10k, w_smd_resistors:r_0805, F.Cu at (33.8, 89.4)
- added SW1: SW_Push, w_switch:PCB_PUSH, F.Cu at (25.9, 97.0)
- added SW2: SW_Push, w_switch:PCB_PUSH, F.Cu at (36.1, 97.0)
- R21, R25, U6: moved to B.Cu
- moved R25 32.2 mm to (49.5, 83.8), turned to 90 degrees
- moved R22 30.5 mm to (58.2, 83.8), turned to 90 degrees
- moved R21 16.0 mm to (48.3, 76.2), turned to 90 degrees
- moved R24 15.6 mm to (54.4, 69.8), turned to 270 degrees
- moved U6 7.73 mm to (50.0, 108.2), turned to 180 degrees
- moved U7 7.08 mm to (50.3, 92.2)
- moved R23 6.84 mm to (43.2, 94.2)
- moved C13 5.84 mm to (71.4, 106.2)
- moved C12 5.33 mm to (65.8, 106.2)
- moved C18 3.97 mm to (55.6, 94.0), turned to 90 degrees
Connections:
- U1 pad 22: Net-(U1-Pad22) -> /BTO1
- U1 pad 23: Net-(U1-Pad23) -> /BTO2
- U1 pad 24: Net-(U1-Pad24) -> +BATT
- U2 pad 3: +BATT -> Net-(U2-Pad3)
Routing:
- net GND: track 0.00 -> 179.3 mm, vias 0 -> 1
- net +5V: track 0.00 -> 128.6 mm, vias 0 -> 1
- net Net-(C4-Pad1): track 0.00 -> 41.7 mm
- net /~MCLR: track 0.00 -> 35.0 mm
- net Net-(J2-Pad1): track 0.00 -> 14.0 mm, vias 0 -> 1
- net /XTAL1: track 0.00 -> 12.0 mm, vias 0 -> 1
- net /XTAL2: track 0.00 -> 11.9 mm, vias 0 -> 1
- net /CAN_H: track 0.00 -> 11.5 mm
- net /CAN_L: track 0.00 -> 11.5 mm
- net Net-(D1-Pad1): track 0.00 -> 8.25 mm
- net /BTO1: track 0.00 -> 7.85 mm
- net /BTO2: track 0.00 -> 7.85 mm
- net /XTAL5: track 0.00 -> 5.64 mm
- net /XTAL6: track 0.00 -> 5.29 mm
- net Net-(C14-Pad1): track 0.00 -> 4.61 mm, vias 0 -> 1
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Other:
- net class PWR added: clearance 0.2, trace_width 0.4, via_dia 0.6, via_drill 0.4

Commit message: placa microchip
Signed-off-by: cuki2 <mauricio@krebs.com.br>
Parts:
- added hole_3mm5: VAL**, w_details:hole_3mm5, F.Cu at (23.0, 23.0)
- added hole_3mm5: VAL**, w_details:hole_3mm5, F.Cu at (23.0, 117.0)
- added hole_3mm5: VAL**, w_details:hole_3mm5, F.Cu at (117.0, 23.0)
- added hole_3mm5: VAL**, w_details:hole_3mm5, F.Cu at (117.0, 117.0)
- C12, C13, Y3: moved to F.Cu
- R3: moved to B.Cu
- moved R14 21.8 mm to (81.5, 71.1), turned to 0 degrees
- moved Q3 17.6 mm to (86.7, 70.6), turned to 270 degrees
- moved D2 5.61 mm to (24.6, 28.4)
- moved R3 5.11 mm to (26.4, 31.2), turned to 90 degrees
- moved C12 3.61 mm to (63.5, 109.0), turned to 180 degrees
- moved Y3 3.45 mm to (67.3, 104.6)
- moved R15 3.05 mm to (81.5, 87.1)
- moved J4 3.00 mm to (104.0, 113.0)
- moved C13 2.81 mm to (71.1, 109.0), turned to 0 degrees
- moved R13 2.79 mm to (84.3, 87.1)
- turned C10 to 0 degrees
- turned D5 to 180 degrees
- turned R8 to 0 degrees
Routing:
- net GND: track 179.3 -> 506.1 mm, vias 1 -> 19
- net +5V: track 128.6 -> 377.6 mm, vias 1 -> 12
- net Net-(C4-Pad1): track 41.7 -> 153.9 mm, vias 0 -> 2
- net /BTO1: track 7.85 -> 109.5 mm, vias 0 -> 5
- net Net-(D10-Pad2): track 0.00 -> 99.5 mm, vias 0 -> 4
- net /TX2: track 0.00 -> 94.1 mm, vias 0 -> 5
- net /TX1: track 0.00 -> 92.7 mm, vias 0 -> 6
- net /BTO2: track 7.85 -> 91.4 mm, vias 0 -> 5
- net /RX2: track 0.00 -> 68.4 mm, vias 0 -> 1
- net Net-(D9-Pad2): track 0.00 -> 57.5 mm, vias 0 -> 4
- net /ENCODER_EN: track 0.00 -> 56.7 mm, vias 0 -> 2
- net +BATT: track 0.00 -> 42.8 mm, vias 0 -> 2
- net /LCD_EN: track 0.00 -> 35.9 mm, vias 0 -> 2
- net Net-(Q3-Pad2): track 0.00 -> 33.3 mm, vias 0 -> 2
- net /LCD_RS: track 0.00 -> 31.3 mm, vias 0 -> 1
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- added copper zone on B.Cu, net GND
- added copper zone on F.Cu, net GND
